File: home_assistant_luefter/platine/esp_luefter_steuerung/esp_luefter_steuerung.kicad_pcb (KiCad board)
At the start: 2 copper layers, 89.5 x 43 mm, 7 parts, among them J1 Conn_01x04_Pin, J2 Conn_01x04_Pin, J3 Conn_01x04_Pin, J4 PWR Input 12V, U1 WeMos_D1_mini, U2 LM7805_TO220

Commit message: increase trace widths
Parts:
- moved J1 22.8 mm to (110.5, 69.5)
- moved J2 6.89 mm to (102.0, 77.5)
Routing:
- net +12V: track 136.9 -> 144.1 mm
- net Net-(J1-Pin_4): track 57.4 -> 63.8 mm
- net GND: track 0.00 -> 0.51 mm
Other:
- board size 89.5 x 43 mm -> 78 x 36 mm
Changed lines of the file:
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@@
 	)
 	(setup
+		(stackup
+			(layer "F.SilkS"
+				(type "Top Silk Screen")
+			)
+			(layer "F.Paste"
+				(type "Top Solder Paste")
+			)
+			(layer "F.Mask"
+				(type "Top Solder Mask")
+				(thickness 0.01)
+			)
+			(layer "F.Cu"
+				(type "copper")
+				(thickness 0.035)
+			)
+			(layer "dielectric 1"
+				(type "core")
+				(thickness 1.51)
+				(material "FR4")
+				(epsilon_r 4.5)
+				(loss_tangent 0.02)
+			)
+			(layer "B.Cu"
+				(type "copper")
+				(thickness 0.035)
+			)
+			(layer "B.Mask"
+				(type "Bottom Solder Mask")
+				(thickness 0.01)
+			)
+			(layer "B.Paste"
+				(type "Bottom Solder Paste")
+			)
+			(layer "B.SilkS"
+				(type "Bottom Silk Screen")
+			)
+			(copper_finish "None")
+			(dielectric_constraints no)
+		)
 		(pad_to_mask_clearance 0)
 		(allow_soldermask_bridges_in_footprints no)
@@
 	(footprint "Connector_PinHeader_2.54mm:PinHeader_1x04_P2.54mm_Vertical"
 		(layer "F.Cu")
-		(at 93.235553 84.387688)
+		(at 110.5 69.5)
 		(descr "Through hole straight pin header, 1x04, 2.54mm pitch, single row")
 		(tags "Through hole pin header THT 1x04 2.54mm single row")
@@
 	(footprint "Connector_PinHeader_2.54mm:PinHeader_1x04_P2.54mm_Vertical"
 		(layer "F.Cu")
-		(at 101.98968 84.387688)
+		(at 101.98968 77.5)
 		(descr "Through hole straight pin header, 1x04, 2.54mm pitch, single row")
 		(tags "Through hole pin header THT 1x04 2.54mm single row")
@@
 	)
 	(gr_rect
-		(start 84.5 60.5)
-		(end 174 103.5)
+		(start 96 64.5)
+		(end 174 100.5)
 		(stroke
 			(width 0.05)
@@
 		(start 161.5 83.340903)
 		(end 153.54545 91.295453)
-		(width 0.2)
+		(width 0.4)
 		(layer "B.Cu")
 		(net 9)
@@
 		(start 144.5 91.28)
 		(end 153.529997 91.28)
-		(width 0.2)
+		(width 0.4)
 		(layer "B.Cu")
 		(net 9)
@@
 		(start 161.5 79.5)
 		(end 161.5 83.340903)
-		(width 0.2)
+		(width 0.4)
 		(layer "B.Cu")
 		(net 9)
 	)
 	(segment
+		(start 101.98968 77.5)
+		(end 102.5 77.5)
+		(width 0.2)
+		(layer "B.Cu")
+		(net 13)
+	)
+	(segment
 		(start 115 96.5)
 		(end 110.5 92)
-		(width 0.2)
+		(width 0.4)
+		(layer "B.Cu")
+		(net 16)
+	)
+	(segment
+		(start 101.98968 85.12)
+		(end 109.98968 77.12)
+		(width 0.4)
 		(layer "B.Cu")
 		(net 16)
@@
 	)
 	(segment
+		(start 109.98968 77.12)
+		(end 110.5 77.12)
+		(width 0.2)
+		(layer "B.Cu")
+		(net 16)
+	)
+	(segment
 		(start 137.8 86.2)
 		(end 127.5 96.5)
-		(width 0.2)
+		(width 0.4)
 		(layer "B.Cu")
 		(net 16)
 	)
 	(segment
-		(start 109.992312 92.007688)
-		(end 101.98968 92.007688)
-		(width 0.2)
+		(start 101.98968 85.12)
+		(end 108.86968 92)
+		(width 0.4)
 		(layer "B.Cu")
 		(net 16)
@@
 		(start 127.5 96.5)
 		(end 115 96.5)
-		(width 0.2)
+		(width 0.4)
 		(layer "B.Cu")
 		(net 16)
@@
 		(start 144.5 86.2)
 		(end 137.8 86.2)
-		(width 0.2)
+		(width 0.4)
 		(layer "B.Cu")
 		(net 16)
@@
 	)
 	(segment
-		(start 93.235553 92.007688)
-		(end 101.98968 92.007688)
-		(width 0.2)
+		(start 108.86968 92)
+		(end 110.5 92)
+		(width 0.4)
 		(layer "B.Cu")
 		(net 16)
@@
 		(start 156.42 78.08)
 		(end 158.5 76)
-		(width 0.2)
+		(width 0.4)
 		(layer "B.Cu")
 		(net 17)
 	)
 	(segment
-		(start 91 98.5)
-		(end 91 89.163241)
-		(width 0.2)
+		(start 107.914892 98.5)
+		(end 98.5 89.085108)
+		(width 0.4)
+		(layer "B.Cu")
+		(net 17)
+	)
+	(segment
+		(start 102.5 80.04)
+		(end 110.5 72.04)
+		(width 0.4)
 		(layer "B.Cu")
 		(net 17)
@@
 		(start 170 78.5)
 		(end 170 83.5)
-		(width 0.2)
+		(width 0.4)
 		(layer "B.Cu")
 		(net 17)
@@
 		(start 158.5 76)
 		(end 167.5 76)
+		(width 0.4)
+		(layer "B.Cu")
+		(net 17)
+	)
+	(segment
+		(start 101.98968 80.04)
+		(end 102.5 80.04)
 		(width 0.2)
 		(layer "B.Cu")
@@
 		(start 167.5 76)
 		(end 170 78.5)
-		(width 0.2)
+		(width 0.4)
 		(layer "B.Cu")
 		(net 17)
@@
 		(start 156.42 79.5)
 		(end 156.42 78.08)
-		(width 0.2)
+		(width 0.4)
 		(layer "B.Cu")
 		(net 17)
 	)
 	(segment
-		(start 155 98.5)
-		(end 91 98.5)
-		(width 0.2)
+		(start 113 86.5)
+		(end 112.5 87)
+		(width 0.4)
 		(layer "B.Cu")
 		(net 17)
 	)
 	(segment
-		(start 101.98968 86.927688)
-		(end 110.492312 86.927688)
+		(start 112.5 87)
+		(end 112.42 86.92)
 		(width 0.2)
 		(layer "B.Cu")
@@
 	)
 	(segment
+		(start 113 74.54)
+		(end 113 86.5)
+		(width 0.4)
+		(layer "B.Cu")
+		(net 17)
+	)
+	(segment
 		(start 170 83.5)
 		(end 155 98.5)
-		(width 0.2)
+		(width 0.4)
 		(layer "B.Cu")
 		(net 17)
 	)
 	(segment
-		(start 91 89.163241)
-		(end 93.235553 86.927688)
-		(width 0.2)
+		(start 110.5 72.04)
+		(end 113 74.54)
+		(width 0.4)
+		(layer "B.Cu")
+		(net 17)
+	)
+	(segment
+		(start 112.42 86.92)
+		(end 110.5 86.92)
+		(width 0.4)
 		(layer "B.Cu")
 		(net 17)
@@
 	)
 	(segment
-		(start 93.235553 86.927688)
-		(end 101.98968 86.927688)
-		(width 0.2)
+		(start 155 98.5)
+		(end 107.914892 98.5)
+		(width 0.4)
+		(layer "B.Cu")
+		(net 17)
+	)
+	(segment
+		(start 98.5 89.085108)
+		(end 98.5 83.52968)
+		(width 0.4)
+		(layer "B.Cu")
+		(net 17)
+	)
+	(segment
+		(start 98.5 83.52968)
+		(end 101.98968 80.04)
+		(width 0.4)
 		(layer "B.Cu")
 		(net 17)
@@
 		(polygon
 			(pts
-				(xy 84.5 60.5) (xy 84.5 103.5) (xy 174 103.5) (xy 174 60.5)
+				(xy 96 64.5) (xy 96 100.5) (xy 174 100.5) (xy 174 64.5)
+			)
+		)
+	)
+	(zone
+		(net 0)
+		(net_name "")
+		(layer "B.Cu")
+		(hatch edge 0.5)
+		(connect_pads
+			(clearance 0)
+		)
+		(min_thickness 0.25)
+		(filled_areas_thickness no)
+		(keepout
+			(tracks not_allowed)
+			(vias not_allowed)
+			(pads not_allowed)
+			(copperpour not_allowed)
+			(footprints allowed)
+		)
+		(placement
+			(enabled no)
+			(sheetname "/")
+		)
+		(fill
+			(thermal_gap 0.5)
+			(thermal_bridge_width 0.5)
+		)
+		(polygon
+			(pts
+				(xy 120 65) (xy 146 65) (xy 146 72) (xy 120 72)
 			)
 		)
